File: fuzz_face/fuzz_face.kicad_pcb (KiCad board)
At the start: 2 copper layers, 15 parts, among them Q1 Q_PNP_EBC, Q2 Q_PNP_EBC

Commit message: Add simple common drain buffer.
Parts:
- removed C1: 2.2u, Capacitor_THT:C_Disc_D9.0mm_W5.0mm_P10.00mm
- removed C2: 20u, Capacitor_THT:C_Disc_D9.0mm_W5.0mm_P10.00mm
- removed C3: 10n, Capacitor_THT:C_Disc_D9.0mm_W5.0mm_P10.00mm
- removed RV1, RV2: R_POT, TerminalBlock:TerminalBlock_bornier-3_P5.08mm
- added C_FUZZ1: 20u, Capacitor_THT:C_Disc_D9.0mm_W5.0mm_P10.00mm, F.Cu at (130.8, 72.4)
- added C_IN1: 2.2u, Capacitor_THT:C_Disc_D9.0mm_W5.0mm_P10.00mm, F.Cu at (113.0, 76.2)
- added C_OUT1: 10n, Capacitor_THT:C_Disc_D9.0mm_W5.0mm_P10.00mm, F.Cu at (113.0, 49.5)
- added RV_FUZZ1: R_POT, TerminalBlock:TerminalBlock_bornier-3_P5.08mm, F.Cu at (120.7, 85.1)
- added RV_VOL1: R_POT, TerminalBlock:TerminalBlock_bornier-3_P5.08mm, F.Cu at (120.7, 57.1)
Routing:
- net Net-(C_FUZZ1-Pad1): track 0.00 -> 13.3 mm
- net Net-(C2-Pad1): track 13.3 -> 0.00 mm
- net Net-(C_OUT1-Pad2): track 0.00 -> 9.78 mm
- net Net-(C3-Pad2): track 9.78 -> 0.00 mm
